File: PCB/PCB Version 0.5/rp2350.kicad_sch (KiCad schematic)
At the start: 24 parts, among them U1 RP2350A, Y1 Crystal_GND24

Commit message: schematics nearly done
Parts:
- added C85, C86: 100n, Capacitor_SMD:C_0402_1005Metric, symbol Device:C
- added U10: W25Q16JVUXIQ, Package_SON:Winbond_USON-8-1EP_3x2mm_P0.5mm_EP0.2x1.6mm, symbol Memory_Flash:W25Q32JVSS
Connections:
- net +3V3: now also C85.1, C86.1, U10.8 (VCC)
- net GND: now also C85.2, C86.2, U10.4 (GND)
- net at U1.55 (QSPI_SD3): now also U10.7 (IO3)
- net at U1.56 (QSPI_SCLK): now also U10.6 (CLK)
- net at U1.57 (QSPI_SD0): now also U10.5 (DI(IO0))
- net at U1.58 (QSPI_SD2): now also U10.3 (IO2)
- net at U1.59 (QSPI_SD1): now also U10.2 (DO(IO1))
- net at U1.60 (QSPI_SS): now also U10.1 (~{CS})
