File: PCB/PCB Version 0.5/ADC.kicad_sch (KiCad schematic)
At the start: 4 parts, among them U9 TLV9002S_RUG_X2QFN

Commit message: wip backup
Parts:
- R26: value 120k -> 100k
Changed lines of the file:
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@@
 			)
 		)
-		(property "Value" "120k"
+		(property "Value" "100k"
 			(at 63.5 33.0199 0)
 			(effects
