File: PCB/PCB Version 0.5/Kolibri v0.5.kicad_sch (KiCad schematic)
At the start: 0 parts

Commit message: schematics nearly done
Other:
- sheet ADC ports: added VBat_HI; removed none
- sheet USB ports: added Curr_ESC, VBat_HI; removed none
- note added: "Overvoltage Protection with TVS-Diodes in USB sheet"
Changed lines of the file:
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@@
 		(color 0 0 0 0)
 	)
+	(junction
+		(at 68.58 138.43)
+		(diameter 0)
+		(color 0 0 0 0)
+	)
 	(bus
 		(pts
@@
 	(wire
 		(pts
+			(xy 68.58 138.43) (xy 68.58 175.26)
+		)
+		(stroke
+			(width 0)
+			(type default)
+		)
+	)
+	(wire
+		(pts
 			(xy 157.48 109.22) (xy 185.42 109.22)
 		)
@@
 		)
 	)
+	(wire
+		(pts
+			(xy 165.1 158.75) (xy 185.42 158.75)
+		)
+		(stroke
+			(width 0)
+			(type default)
+		)
+	)
 	(bus
 		(pts
@@
 		)
 	)
+	(wire
+		(pts
+			(xy 162.56 172.72) (xy 162.56 156.21)
+		)
+		(stroke
+			(width 0)
+			(type default)
+		)
+	)
 	(bus
 		(pts
@@
 		)
 	)
+	(wire
+		(pts
+			(xy 68.58 175.26) (xy 165.1 175.26)
+		)
+		(stroke
+			(width 0)
+			(type default)
+		)
+	)
 	(bus
 		(pts
@@
 		)
 	)
+	(wire
+		(pts
+			(xy 165.1 175.26) (xy 165.1 158.75)
+		)
+		(stroke
+			(width 0)
+			(type default)
+		)
+	)
 	(bus
 		(pts
@@
 		)
 	)
+	(wire
+		(pts
+			(xy 71.12 140.97) (xy 81.28 140.97)
+		)
+		(stroke
+			(width 0)
+			(type default)
+		)
+	)
 	(bus
 		(pts
@@
 		)
 	)
+	(wire
+		(pts
+			(xy 162.56 156.21) (xy 185.42 156.21)
+		)
+		(stroke
+			(width 0)
+			(type default)
+		)
+	)
 	(bus
 		(pts
@@
 		)
 	)
+	(wire
+		(pts
+			(xy 71.12 172.72) (xy 162.56 172.72)
+		)
+		(stroke
+			(width 0)
+			(type default)
+		)
+	)
 	(bus
 		(pts
@@
 	(wire
 		(pts
+			(xy 71.12 140.97) (xy 71.12 172.72)
+		)
+		(stroke
+			(width 0)
+			(type default)
+		)
+	)
+	(wire
+		(pts
 			(xy 105.41 120.65) (xy 130.81 120.65)
 		)
@@
 			(width 0)
 			(type default)
+		)
+	)
+	(text "Overvoltage Protection with TVS-Diodes in USB sheet"
+		(exclude_from_sim no)
+		(at 116.332 174.244 0)
+		(effects
+			(font
+				(size 1.27 1.27)
+			)
 		)
 	)
 	(label "Motor{[1..4]}"
 		(at 109.22 71.12 0)
-		(fields_autoplaced yes)
 		(effects
 			(font
@@
 	(label "I2C0{SDA SCL}"
 		(at 109.22 81.28 0)
-		(fields_autoplaced yes)
 		(effects
 			(font
@@
 	(label "SPI0{SCLK SDX}"
 		(at 161.29 130.81 0)
-		(fields_autoplaced yes)
 		(effects
 			(font
@@
 	(label "USB{D+ D-}"
 		(at 162.56 153.67 0)
-		(fields_autoplaced yes)
 		(effects
 			(font
@@
 	(label "U0{TX RX}"
 		(at 109.22 68.58 0)
-		(fields_autoplaced yes)
 		(effects
 			(font
@@
 	(label "Video{In Out}"
 		(at 153.67 40.64 0)
-		(fields_autoplaced yes)
 		(effects
 			(font
@@
 	(label "SPI1{MISO SCLK MOSI}"
 		(at 161.29 80.01 0)
-		(fields_autoplaced yes)
 		(effects
 			(font
@@
 	(label "PWM{[1..4]}"
 		(at 109.22 50.8 0)
-		(fields_autoplaced yes)
 		(effects
 			(font
@@
 	(label "U2{TX RX}"
 		(at 109.22 78.74 0)
-		(fields_autoplaced yes)
 		(effects
 			(font
@@
 	(label "SD_DAT{[0..3]}"
 		(at 161.29 106.68 0)
-		(fields_autoplaced yes)
 		(effects
 			(font
@@
 	(label "ADC{Curr VBat}"
 		(at 111.76 138.43 0)
-		(fields_autoplaced yes)
 		(effects
 			(font
@@
 	(label "U1{TX RX}"
 		(at 109.22 73.66 0)
-		(fields_autoplaced yes)
 		(effects
 			(font
@@
 	(label "Spk{+ -}"
 		(at 73.66 111.76 90)
-		(fields_autoplaced yes)
 		(effects
 			(font
@@
 	(label "{SWDIO SWCLK}"
 		(at 109.22 76.2 0)
-		(fields_autoplaced yes)
 		(effects
 			(font
@@
 	(sheet
 		(at 81.28 135.89)
-		(size 24.13 5.08)
+		(size 24.13 7.62)
 		(fields_autoplaced yes)
 		(stroke
@@
 		)
 		(property "Sheetfile" "ADC.kicad_sch"
-			(at 81.28 141.5546 0)
+			(at 81.28 144.0946 0)
 			(effects
 				(font
@@
 		(pin "Curr_ESC" input
 			(at 81.28 138.43 180)
+			(effects
+				(font
+					(size 1.27 1.27)
+				)
+				(justify left)
+			)
+		)
+		(pin "VBat_HI" output
+			(at 81.28 140.97 180)
 			(effects
 				(font
@@
 	(sheet
 		(at 185.42 151.13)
-		(size 22.86 5.08)
+		(size 22.86 10.16)
 		(fields_autoplaced yes)
 		(stroke
@@
 		)
 		(property "Sheetfile" "usb.kicad_sch"
-			(at 185.42 156.7946 0)
+			(at 185.42 161.8746 0)
 			(effects
 				(font
@@
 			(effects
 				(font
+					(size 1.27 1.27)
+				)
+				(justify left)
+			)
+		)
+		(pin "VBat_HI" input
+			(at 185.42 156.21 180)
+			(effects
+				(font
+					(size 1.27 1.27)
+				)
+				(justify left)
+			)
+		)
+		(pin "Curr_ESC" input
+			(at 185.42 158.75 180)
+			(effects
+				(font
