File: PCB/PCB Version 0.5/connectors.kicad_sch (KiCad schematic)
At the start: 38 parts, among them J5 Conn_01x08_MountingPin, J6 Conn_01x06_MountingPin, J7 Conn_01x06_MountingPin, J8 Conn_01x03_MountingPin

Commit message: wip routing
Connections:
- net GND: now also J6.MP (MountPin)
- net U1.RX: now also P6.1; no longer P7.1
- net U1.TX: now also P7.1; no longer P6.1
Changed lines of the file:
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@@
 		)
 	)
+	(label "U1.RX"
+		(at 36.83 119.38 0)
+		(effects
+			(font
+				(size 1.27 1.27)
+			)
+			(justify left bottom)
+		)
+	)
 	(label "U2.RX"
 		(at 36.83 172.72 0)
@@
 		)
 	)
-	(label "U1.TX"
-		(at 36.83 119.38 0)
-		(effects
-			(font
-				(size 1.27 1.27)
-			)
-			(justify left bottom)
-		)
-	)
 	(label "U0.TX"
 		(at 148.59 57.15 0)
@@
 		)
 	)
-	(label "U1.RX"
-		(at 36.83 121.92 0)
-		(effects
-			(font
-				(size 1.27 1.27)
-			)
-			(justify left bottom)
-		)
-	)
 	(label "Spk.-"
 		(at 148.59 124.46 0)
@@
 		)
 	)
+	(label "U1.TX"
+		(at 36.83 121.92 0)
+		(effects
+			(font
+				(size 1.27 1.27)
+			)
+			(justify left bottom)
+		)
+	)
 	(label "I2C0.SDA"
 		(at 58.42 105.41 0)
@@
 					(unit 1)
 				)
+			)
+		)
+	)
+	(symbol
+		(lib_id "power:GND")
+		(at 76.2 113.03 0)
+		(unit 1)
+		(exclude_from_sim no)
+		(in_bom yes)
+		(on_board yes)
+		(dnp no)
+		(fields_autoplaced yes)
+		(property "Reference" "#PWR0172"
+			(at 76.2 119.38 0)
+			(effects
+				(font
+					(size 1.27 1.27)
+				)
+				(hide yes)
+			)
+		)
+		(property "Value" "GND"
+			(at 76.2 118.11 0)
+			(effects
+				(font
+					(size 1.27 1.27)
+				)
+			)
+		)
+		(property "Footprint" ""
+			(at 76.2 113.03 0)
+			(effects
+				(font
+					(size 1.27 1.27)
+				)
+				(hide yes)
+			)
+		)
+		(property "Datasheet" ""
+			(at 76.2 113.03 0)
+			(effects
+				(font
+					(size 1.27 1.27)
+				)
+				(hide yes)
+			)
+		)
+		(property "Description" "Power symbol creates a global label with name \"GND\" , ground"
+			(at 76.2 113.03 0)
+			(effects
+				(font
+					(size 1.27 1.27)
+				)
+				(hide yes)
+			)
+		)
+		(pin "1"
+		)
+		(instances
+			(project ""
+				(path "/1651f454-30c0-48ea-9fcf-6c96a661786a/c061bb86-7a8e-4300-a3f9-744e498f6d03"
+					(reference "#PWR0172")
+					(unit 1)
+				)
