File: PCB/PCB Version 0.5/sd.kicad_sch (KiCad schematic)
At the start: 3 parts, among them J9 Micro_SD_Card_Det1

Commit message: wip backup
Parts:
- C74, C75: footprint Capacitor_SMD:C_0402_1005Metric -> Capacitor_SMD:C_0402_1005Metric_Pad0.74x0.62mm_HandSolder
Changed lines of the file:
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@@
 			)
 		)
-		(property "Footprint" "Capacitor_SMD:C_0402_1005Metric"
+		(property "Footprint" "Capacitor_SMD:C_0402_1005Metric_Pad0.74x0.62mm_HandSolder"
 			(at 86.0552 95.25 0)
 			(effects
@@
 			)
 		)
-		(property "Footprint" "Capacitor_SMD:C_0402_1005Metric"
+		(property "Footprint" "Capacitor_SMD:C_0402_1005Metric_Pad0.74x0.62mm_HandSolder"
 			(at 73.3552 95.25 0)
 			(effects

Commit message: wip routing
Connections:
- net SD_DAT.3: no longer J9.8 (DAT1)
- new net SD_DAT.1: J9.8 (DAT1)
Changed lines of the file:
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@@
 		)
 	)
-	(label "SD_DAT.3"
+	(label "SD_DAT.1"
 		(at 156.21 93.98 0)
 		(effects
