File: PCB/PCB Version 0.5/_autosave-Kolibri v0.5.kicad_pcb (KiCad board)
At the start: 8 copper layers, 38 x 38 mm, 216 parts, among them IC1 SX1280IMLTRT, IC2 RFX2401C, IC3 SX1280IMLTRT, IC4 RFX2401C, IC5 LMR38025SDRRR, IC6 LMR38025SDRRR, J1 USB_C_Receptacle_USB2.0_16P, J2 Conn_01x04_MountingPin, J3 Conn_Coaxial_Small, J4 Conn_Coaxial_Small, J5 Conn_01x08_MountingPin, J6 Conn_01x06_MountingPin, J7 Conn_01x06_MountingPin, J8 Conn_01x03_MountingPin, J9 Micro_SD_Card_Det1, Q1 BSS138, U1 RP2350A, U10 W25Q16JVUXIQ, U11 LPS22HB, U2 BMI270, U3 ESP32-U4WDH, U4 TPS2116DRL, U5 AT7456E, U6 LP5912-3.3DRV, U7 TPS746-3.3DRV, U8 WE-TVS-824015043, U9 TLV9002S_RUG_X2QFN, Y1 Crystal_GND24, Y2 Crystal_GND24, Y3 Crystal_GND24, Y4 Crystal_GND24, Y5 Crystal_GND24

Commit message: backup before recovery
Routing:
- net /ELRS/ELRS_BUTTON: track 0.00 -> 10.0 mm, vias 0 -> 1
- net /ELRS/RADIO_RST_2: track 0.00 -> 4.26 mm, vias 0 -> 1
- net /PWM.4: track 0.00 -> 3.03 mm, vias 0 -> 1
- net +3V3_ELRS: track 19.2 -> 22.0 mm, vias 12 -> 13
- net /ELRS/RADIO_BUSY_2: track 0.00 -> 2.24 mm, vias 0 -> 1
- net /ELRS/RADIO_DIO1_2: track 0.00 -> 1.76 mm
- net /ELRS/RADIO_MISO: track 0.00 -> 1.40 mm
- net /ELRS/RADIO_DIO1: track 0.00 -> 1.36 mm, vias 0 -> 1
- net /ELRS/POWER_RXEN2: track 0.00 -> 1.35 mm, vias 0 -> 1
- net /ELRS/RADIO_MOSI: track 0.00 -> 1.04 mm
- net /ELRS/RADIO_RST: track 0.00 -> 1.01 mm, vias 0 -> 1
- net /ELRS/POWER_TXEN_2: track 1.63 -> 2.51 mm, vias 1 -> 2
- net /ELRS/RADIO_NSS: track 0.00 -> 0.86 mm, vias 0 -> 1
- net /PWM.3: track 0.00 -> 0.84 mm, vias 0 -> 1
- net /PWM.2: track 0.00 -> 0.68 mm, vias 0 -> 1
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