File: PCB/PCB Version 0.5/ELRS.kicad_sch (KiCad schematic)
At the start: 59 parts, among them IC1 SX1280IMLTRT, IC2 RFX2401C, IC3 SX1280IMLTRT, IC4 RFX2401C, J3 Conn_Coaxial_Small, J4 Conn_Coaxial_Small, U3 ESP32-U4WDH, Y2 Crystal_GND24, Y3 Crystal_GND24, Y5 Crystal_GND24

Commit message: 0 DRC violations/warnings 🎉
Connections:
- net POWER_RXEN2 is gone; now on net POWER_RXEN_2: U3.34 (GPIO5/S1)
- net PWM.3: now also U3.39 (GPIO22); no longer U3.36 (GPIO23)
- net PWM.4: now also U3.36 (GPIO23); no longer U3.39 (GPIO22)
Changed lines of the file:
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@@
+			"AAAAAAAAAAAAAAAAAAAAAAAAAAAAAAAAAAAAAAAAAAAAAAAAAAAAAAAAAAAAAAAAAAAAAAAAAAAA"
+			"AAAAAAAAAAAAAAAAAAAAAAAAAAAAAAAAAAAAAAAAAAAAAAAAAAAAAAAAAAAAAAAAAAAAAAAAAAAA"
+			"AAAAAAAAAAAAAAAAAAAAAAAAAAAAAAAAAAAAAAAAAAAAAAAAAAAAAAAAAAAAAAAAAAAAAAAAAAAA"
+			"AAAAAAAAAAAAAAAAAAAAAAAAAAAAAAAAAAAAAAAAAAAAAAAAAAAAAAAAAAAAAAAAAAAAAAAAAAAA"
+			"AAAAAAAAAAAAAAAAAAAAAAAAAAAAAAAAAAAAAAAAAAAAAAAAAAAAAAAAAAAAAAAAAAAAAAAAAAAA"
+			"AAAAAAAAAAAAAAAAAAAAAAAAAAAAAAAAAAAAAAAAAAAAAAAAAAAAAAAAAAAAAAAAAAAAAAAAAAAA"
+			"AAAAAAAAAAAAAAAAAAAAAAAAAAAAAAAAAAAAAAAAAAAAAAAAAAAAAAAAAAAAAAAAAAAAAAAAAAAA"
+			"AAAAAAAAAAAAAAAAAAAAAAAAAAAAAAAAAAAAAAAAAAAAAAAAAAAAAAAAAAAAAAAAAAAAAAAAAAAA"
+			"AAAAAAAAAAAAAAAAAAAAAAAAAAAAAAAAAAAAAAAAAAAAAAAAAAAAAAAAAAAAAAAAAAAAAAAAAAAA"
+			"AAAAAAAAAAAAAAAAAAAAAAAAAAAAAAAAAAAAAAAAAAAAAAAAAAAAAAAAAAAAAAAAAAAAAAAAAAAA"
+			"AAAAAAAAAAAAAAAAAAAAAAAAAAAAAAAAAAAAAAAAAAAAAAAAAAAAAAAAAAAAAAAAAAAAAAAAAAAA"
+			"AAAAAAAAAAAAAAAAAAAAAAAAAAAAAAAAAAAAAAAAAAAAAAAAAAAAAAAAAAAAAAAAAAAAAAAAAAAA"
+			"AAAAAAAAAAAAAAAAAAAAAAAAAAAAAAAAAAAAAAAAAAAAAAAAAAAAAAAAAAAAAAAAAAAAAAAAAAAA"
+			"AAAAAAAAAAAAAAAAAAAAAAAAAAAAAAAAAAAAAAAAAAAAAAAAAAAAAAAAAAAAAAAAAAAAAAAAAAAA"
+			"AAAAAAAAAAAAAAAAAAAAAAAAAAAAAAAAAAAAAAAAAAAAAAAAAAAAAAAAAAAAAAAAAAAAAAAAAAAA"
+			"AAAAAAAAAAAAAAAAAAAAAAAAAAAAAAAAAAAAAAAAAAAAAAAAAAAAAAAAAAAAAAAAAAAAAAAAAAAA"
+			"AAAAAAAAAAAAAAAAAAAAAAAAAAAAAAAAAAAAAAAAAAAAAAAAAAAAAAAAAAAAAAAAAAAAAAAAAAAA"
+			"AAAAAAAAAAAAAAAAAAAAAAAAAAAAAAAAAAAAAAAAAAAAAAAAAAAAAAAAAAAAAAAAAAAAAAAAAAAA"
 			"AAAAAAAAAAAAAAAAAAAAAAAAAAAAAAAAAAAAAAAAAAAAAAAAAAAAAAAAAAAAAAAAAAAAAAAAAAAA"
 			"AAAAAAAAAAAAAAAAAAAAAAAAAAAAAAAAAAAAAAAAAAAAAAAAAAAAAAAAAAAAAAAAAAAAAAAAAAAA"
@@
 			"////////////////////////////////////////////////////////////////////////////"
 			"////////////////////////////////////////////////////////////////////////////"
+			"////////////////////////////////////////////////////////////////////////////"
+			"////////////////////////////////////////////////////////////////////////////"
+			"////////////////////////////////////////////////////////////////////////////"
+			"////////////////////////////////////////////////////////////////////////////"
+			"////////////////////////////////////////////////////////////////////////////"
+			"////////////////////////////////////////////////////////////////////////////"
+			"////////////////////////////////////////////////////////////////////////////"
+			"////////////////////////////////////////////////////////////////////////////"
+			"////////////////////////////////////////////////////////////////////////////"
+			"////////////////////////////////////////////////////////////////////////////"
+			"////////////////////////////////////////////////////////////////////////////"
+			"////////////////////////////////////////////////////////////////////////////"
+			"//////////////////////////////////////////////////////////+3V/8PL4f/1///////"
+			"////////////////////////////////1/+HLw//V7f/////////////////////////////////"
+			"/+eXP/8HR5//7////7dfD/8nd8//////////////////////////////////////////z/93Jxf/"
+			"X7f//////////////////////////////////+eXN/8PV7f/////////9/+/Xxf/F0eH/7/n9///"
+			"//////////////////////////////////////////////////////////evT/8PP5f/5///////"
+			"////////////////////55f/PwdH/6f3////////55c3/w9Xt//////////3/79fF/8XR4f/v+f3"
 			"/////////////////////////w=="
 		)
@@
 			"////////////////////////////////////////////////////////////////////////////"
 			"////////////////////////////////////////////////////////////////////////////"
+			"////////////////////////////////////////////////////////////////////////////"
+			"////////////////////////////////////////////////////////////////////////////"
+			"////////////////////////////////////////////////////////////////////////////"
+			"//////////////////////////////////////////////////////////////////+YmJj/Z2dn"
+			"////////////////////////////////////////////////////////////////////////////"
+			"////////////////////////////////////////////////////////////////////////////"
+			"////////////////z3f/Jx9n/8f/////////////////////////////////v/9nFy//d9f/////"
+			"////////////////////////////////////////////////////////////////////////////"
+			"////////////////////////////////////////////////////////////////////////////"
+			"//////////84ODj/x8fH////////////////////////////////////////////////////////"
+			"////////////////////////////////////////////////////////////////////////////"
+			"///////////////////////////////////w8PD/Dw8P////////////////////////////////"
+			"//////////////////////////////////+3V/8PL4f/1///////////////////////////////"
+			"14cv/w8/l//n///////3/6dPB/9Hn+///////++/j/9nl8///////////////////////+/Hd/8v"
+			"D0f/n+f/////x/9nHxf/V6/v////////////////////1/93Lx//Z7//////////z3f/Jxdf/7//"
+			"///////////////////////////H/28fH/9vx////////+eXN/8PV7f/////////1/93Jxf/X7/3"
+			"////////////////////////////////////////////759H/w8/n//n////////////////////"
+			"///////nl/8/B0f/p/f/////////////////////////////////////////////////////////"
 			"/////////////////////////w=="
 		)
@@
 			"////////////////////////////////////////////////////////////////////////////"
 			"////////////////////////////////////////////////////////////////////////////"
-			"/////////////////////////////////////////////////////////w=="
+			"/////////////////////////////////////////////////////////wAAAAAAAAAAAAAAAAAA"
+			"AAAAAAAAAAAAAAAAAAAAAAAAAAAAAAAAAAAAAAAAAAAAAAAAAAAAAAAAAAAAAAAAAAAAAAAAAAAA"
+			"AAAAAAAAAAAAAAAAAAAAAAAAAAAAAAAAAAAAAAAAAAAAAAAAAAAAAAAAAAAAAAAAAAAAAAAAAAAA"
+			"AAAAAAAAAAAAAAAAAAAAAAAAAAAAAAAAAAAAAAAAAAAAAAAAAAAAAAAAAAAAAAAAAAAAAAAA7e3t"
+			"ABwcHAAAAAAAAAAAAAAAAAAAAAAAAAAAAAAAAAAAAAAAAAAAAAAAAAAAAAAAAAAAAAAAAAAAAAAA"
+			"AAAAAAAAAAAAAAAAAAAAAAAAAAAAAAAAAAAAAAAAAAAAAAAAAAAAAAAAAAAAAAAAAAAAAAAAAAAA"
+			"AAAAAAAAAAAAAAAAAAAAAAAAAAAAAAAAAAAAAAAAAAQAAAAAAAAAAAAAAAAAAAAAAAAAAAAAAAAA"
+			"AAAAAAAAAAAAAAAAAAAAAAAAAAAAAAAAAAAAAAAAAAAAAAAAAAAAAAAAAAAAAAAAAAAAAAAAAAAA"
+			"AAAAAAAAAAAAAAAAAAAAAAAAAAAAAAAAAAAAAAAAAAAAAAAAAABHR0cAAgICAAAAAAAAAAAAAAAA"
+			"AAAAAAAAAAAAAAAAAAAAAAAAAAAAAAAAAAAAAAAAAAAAAAAAAAAAAAAAAAAAAAAAAAAAAAAAAAAA"
+			"AAAAAAAAAAAAAAAAAAAAAAAAAAAAAAAAAAAAAAAAAAAAAAAAAAAAAAAAAAAAAAAAAAAAAAAAAAAA"
+			"AAAAAAAAAAAAAAAAAAAAAAAAAAAAAAAAAAAAAAAAAAAAAAAAAAAAAAAAAAAAAAAAAAAAAAAAAAAA"
+			"AAAAAAAAAAAAAAAAAAAAAAAAAAAAAAAAAAAAAAAAAAAAAAAAAAAAAAAAAAAAAAAAAAAAAAAAAAAA"
+			"AAAAAAAAAAAAAAAAAAAAAAAAAAAAAAAAAAAAAAAAAAAAAAAAAAAAAAAAAAAAAAAAAAAAAAAAAAAA"
+			"AAAAAAAAAAAAAAAAAAAAAAAAAAAAAAAAAAAAAAAAAAAAAAAAAAAAAAAAAAAAAAAAAAAAAAAAAAAA"
+			"AAAAAAAAAAAAAAAAAAAAAAAAAAAAAAAAAAAAAAAAAAAAAAAAAAAAAAAAAAAAAAAAAAAAAAAAAAAA"
+			"AAAAAAAAAAAAAAAAAAAAAAAAAAAAAAAAAAAAAAAAAAAAAAAAAAAAAAAAAAAAAAAAAAAAAAAAAAAA"
+			"AAAAAAAAAAAAAAAAAAAAAAAAAAAAAAAAAAAAAAAAAAAAAAAAAAAAAAAAAAAAAAAAAAAAAAAAAAAA"
+			"AAAAAAAAAAAAAAAAAAAAAAAAAAAAAAAAAAAAAAAAAAAAAAAAAAAAAAAAAA=="
 		)
 	)
@@
 			"T29HUExpdGtYMzRmL2pXTjcrT2F0aDQ3WkJjMVU2L09BQjFUVHM2NlFPZ29xbDFvS1FzZ1RRaGZR"
 			"MUxsbzA1bFEvUWRmUjZkZUcwUEV2NUF2ajBCOTg4TnBYLzYzLytNYTloMURsSVNWSkFNN0dPcmxj"
-			"ak9zYlVzcFE0QXpUcmVGNUZ4NXhjbGlWa3I0R24zK01ibA=="
+			"ak9zYlVzcFE0QXpUcmVGNUZ4NXhjbGlWa3I0R24zK01ibGZKcmYvaC8rQVI0bldVbmRob1V0MGR3"
+			"YndNMS9TbmYrLy8va0Z1cWdkUHNFaFhxVWR3VUhjdjE4SXdNdjl2RXRYVFVyLzkvdEU4WW9LNm9r"
+			"N1dpb0NoQVhSMytlN2hZbVZsM3grc0xNQ3pNWlhpZEpXVFZ0Rk1jLzY1SzNTOFM1emVoVnNzL1Ry"
+			"YnRDZFdZbjZ0dEYyVHA1NENCYlIydkJjMnkwWUFzVHF0SjU2U2lqYWV6VGl5emJBUDRuSFRVd1pV"
+			"azZlSmQ0YW51cTl4N2tkSTFvQXc5OUcvOWxGZWFRN3Zsbk5qeEFVQzFhSVVaWGhveUdBUUUvb0Nm"
+			"L3Q4LzU2ZTlEdHRCaU8vcTFUWGVvdUdKYm5YckFlMFRCcVVwaGc3a293dnVCUnVkWit2cmQrZzFy"
+			"ZGtYVE5XaWVwMDVvdUYwSS9KMlFoZ0UrTUdBOENjLzRPT2ZkRm03R3hEMUhGUks0cTZEKzRPbnZL"
+			"b3ZzMm83TkI4MjhGUWY2ODgvckg3aHVieXVMcmpHenVoYkRNbTJmYkp6dCszVHpmdytTWkt1clN2"
+			"YytUbWlPQjA2R3dIZmY5cWxGWGlFaDg5VEtvcVlYcnRMcExZSXVnNWUyOEZyUXg1M2NaMGY4Rk92"
+			"UXlQM2g0OW4zb1JoWXRUaDR6Z2l3Wm4raFp4bHcxK2VwOUFNZ3lVK29WUXRHbDdsQkYxa1pPam9L"
+			"b0NPYWNDSGFVS2NVN21ya0kwZXc0d1pXUHFjZVhVTG8vNWpQaTkxYk0vRG1FaUNuQ3hUMFE5dndW"
+			"ZmxoTjAyL2NTa0U3UndtaVpPczB1WmhiUmNsNS84dUVuSHkraHBQdTNPVTE2dDN1RkoxTWNlYlU4"
+			"WitpYytjbmhqV1VKR1k3b2UwcGprRmRRM3pOTTd5UXRiSU02WFFiYnQwL09lcTIycjZNWUtmSndT"
+			"eFFXdDRZWWV5dU9ZRERDczhiY3F3R3ZLb29ESjdsUlJ6SjZ0ZHFLY0xDM0FuQ3l2SUE1VFlCbkRV"
+			"SUVDaFRwUWtGZSt2TGllYjdLVXBDdmhDai8ybXFUamRadXM4Z1VmdHp1YzhBUUZsSkowOEhOKzNt"
+			"dlRuM2cvdm1aYUdDcFFMdmkyM0NyVnhYT1c0TE0relc1OGRLSXJVM3F0THA5TzVwMUJzVDBhSy9D"
+			"NTM2SVRUNXk0eW9TdVkvS0hSb01nQnpCd3ZUWHFyNS9TOGZva2h4dGRFTGRiOUQ4L1doVjBYRzg0"
+			"SnVITXZLcEQwMW1DVDdzMCs2TTNIby95UmkwSHd6Qm9uaHhjeW5qQXp6L3Mwdkd6bzZXNmhhMHJR"
+			"RWxaQUVWRy9ocnFoajF4c2NvSSt0SEYzNm41ckRkZEQwVg=="
 		)
 	)
@@
 		)
 	)
-	(label "POWER_RXEN2"
+	(label "POWER_RXEN_2"
 		(at 212.09 151.13 180)
 		(effects
@@
 		)
 	)
-	(label "PWM.3"
+	(label "PWM.4"
 		(at 212.09 185.42 180)
 		(effects
@@
 		)
 	)
-	(label "PWM.4"
+	(label "PWM.3"
 		(at 212.09 182.88 180)
 		(effects
